File: solene.sch (EAGLE design)
At the start: 1 part, among them J1X CLONOLU

Commit message: rev 1
Parts:
- added D1: 1N4004, diode:DIODE-D-2.5
- added JP1: (no value), SparkFun-Passives:JUMPER-2PTH
- added Q2: IRF540, transistor-power:IRF540
- added R1: 2k2, rcl:R-US_0204/2V
Connections:
- new net N$1: J1XA4983$1.STEP, JP1.1
- new net N$2: JP1.2, R1.1
- new net N$3: Q2.G, R1.2
- new net N$4: D1.C, J1XA4983$2.2B, J1XA4983$2.VMOT
- new net N$5: D1.A, J1XA4983$2.2A, Q2.D
- net GND: now also Q2.S
Changed lines of the file:
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@@
 <layer number="19" name="Unrouted" color="6" fill="1" visible="no" active="no"/>
 <layer number="20" name="Dimension" color="15" fill="1" visible="no" active="no"/>
-<layer number="21" name="tPlace" color="7" fill="1" visible="no" active="no"/>
-<layer number="22" name="bPlace" color="7" fill="1" visible="no" active="no"/>
+<layer number="21" name="tPlace" color="16" fill="1" visible="no" active="no"/>
+<layer number="22" name="bPlace" color="14" fill="1" visible="no" active="no"/>
 <layer number="23" name="tOrigins" color="15" fill="1" visible="no" active="no"/>
 <layer number="24" name="bOrigins" color="15" fill="1" visible="no" active="no"/>
@@
 <layer number="49" name="Reference" color="7" fill="1" visible="no" active="no"/>
 <layer number="50" name="dxf" color="7" fill="1" visible="no" active="no"/>
-<layer number="51" name="tDocu" color="7" fill="1" visible="no" active="no"/>
+<layer number="51" name="tDocu" color="6" fill="1" visible="no" active="no"/>
 <layer number="52" name="bDocu" color="7" fill="1" visible="no" active="no"/>
 <layer number="53" name="tGND_GNDA" color="7" fill="9" visible="no" active="no"/>
@@
 <layer number="97" name="Info" color="7" fill="1" visible="yes" active="yes"/>
 <layer number="98" name="Guide" color="6" fill="1" visible="yes" active="yes"/>
+<layer number="99" name="SpiceOrder" color="5" fill="1" visible="yes" active="yes"/>
 <layer number="100" name="Muster" color="7" fill="1" visible="no" active="no"/>
 <layer number="101" name="Patch_Top" color="12" fill="4" visible="yes" active="yes"/>
@@
 <layer number="106" name="bPlate" color="7" fill="1" visible="yes" active="yes"/>
 <layer number="107" name="Crop" color="7" fill="1" visible="yes" active="yes"/>
+<layer number="108" name="tplace-old" color="10" fill="1" visible="yes" active="yes"/>
+<layer number="109" name="ref-old" color="11" fill="1" visible="yes" active="yes"/>
 <layer number="116" name="Patch_BOT" color="9" fill="4" visible="yes" active="yes"/>
 <layer number="121" name="_tsilk" color="7" fill="1" visible="yes" active="yes"/>
 <layer number="122" name="_bsilk" color="7" fill="1" visible="yes" active="yes"/>
+<layer number="125" name="_tNames" color="7" fill="1" visible="no" active="yes"/>
+<layer number="144" name="Drill_legend" color="7" fill="1" visible="no" active="yes"/>
 <layer number="151" name="HeatSink" color="7" fill="1" visible="yes" active="yes"/>
+<layer number="199" name="Contour" color="7" fill="1" visible="yes" active="yes"/>
 <layer number="200" name="200bmp" color="1" fill="10" visible="yes" active="yes"/>
 <layer number="201" name="201bmp" color="2" fill="10" visible="yes" active="yes"/>
@@
 <layer number="207" name="207bmp" color="8" fill="10" visible="yes" active="yes"/>
 <layer number="208" name="208bmp" color="9" fill="10" visible="yes" active="yes"/>
+<layer number="209" name="209bmp" color="7" fill="1" visible="no" active="yes"/>
+<layer number="210" name="210bmp" color="7" fill="1" visible="no" active="yes"/>
+<layer number="211" name="211bmp" color="7" fill="1" visible="no" active="yes"/>
+<layer number="212" name="212bmp" color="7" fill="1" visible="no" active="yes"/>
+<layer number="213" name="213bmp" color="7" fill="1" visible="no" active="yes"/>
+<layer number="214" name="214bmp" color="7" fill="1" visible="no" active="yes"/>
+<layer number="215" name="215bmp" color="7" fill="1" visible="no" active="yes"/>
+<layer number="216" name="216bmp" color="7" fill="1" visible="no" active="yes"/>
+<layer number="217" name="217bmp" color="18" fill="1" visible="no" active="no"/>
+<layer number="218" name="218bmp" color="19" fill="1" visible="no" active="no"/>
+<layer number="219" name="219bmp" color="20" fill="1" visible="no" active="no"/>
+<layer number="220" name="220bmp" color="21" fill="1" visible="no" active="no"/>
+<layer number="221" name="221bmp" color="22" fill="1" visible="no" active="no"/>
+<layer number="222" name="222bmp" color="23" fill="1" visible="no" active="no"/>
+<layer number="223" name="223bmp" color="24" fill="1" visible="no" active="no"/>
+<layer number="224" name="224bmp" color="25" fill="1" visible="no" active="no"/>
 <layer number="250" name="Descript" color="3" fill="1" visible="no" active="no"/>
 <layer number="251" name="SMDround" color="12" fill="11" visible="no" active="no"/>
@@
 <parts>
 <part name="J1X" library="pololu-allegro" deviceset="CLONOLU" device=""/>
-<part name="GND37" library="SparkFun" deviceset="GND" device=""/>
 <part name="GND38" library="SparkFun" deviceset="GND" device=""/>
-<part name="U$26" library="pwr" deviceset="VDD" device=""/>
-<part name="U$27" library="pwr" deviceset="VMOT" device=""/>
+<part name="JP1" library="SparkFun-Passives" deviceset="JUMPER-2" device="PTH"/>
+<part name="Q2" library="transistor-power" deviceset="IRF540" device=""/>
+<part name="D1" library="diode" deviceset="DIODE-" device="D-2.5" value="1N4004"/>
+<part name="R1" library="rcl" deviceset="R-US_" device="0204/2V" value="2k2"/>
 </parts>
 <sheets>
@@
 </plain>
 <instances>
-<instance part="J1X" gate="A4983$1" x="-137.16" y="-55.88"/>
-<instance part="J1X" gate="A4983$2" x="-137.16" y="60.96"/>
-<instance part="GND37" gate="1" x="-149.86" y="45.72"/>
-<instance part="GND38" gate="1" x="-119.38" y="45.72"/>
-<instance part="U$26" gate="G$1" x="-111.76" y="55.88"/>
-<instance part="U$27" gate="G$1" x="-162.56" y="55.88"/>
+<instance part="J1X" gate="A4983$1" x="-144.78" y="50.8" rot="R270"/>
+<instance part="J1X" gate="A4983$2" x="-68.58" y="50.8" rot="R270"/>
+<instance part="GND38" gate="1" x="-81.28" y="25.4"/>
+<instance part="JP1" gate="A" x="-132.08" y="40.64"/>
+<instance part="Q2" gate="G$1" x="-109.22" y="40.64"/>
+<instance part="D1" gate="G$1" x="-96.52" y="55.88" rot="R90"/>
+<instance part="R1" gate="G$1" x="-121.92" y="38.1"/>
 </instances>
 <busses>
@@
 <pinref part="GND38" gate="1" pin="GND"/>
 <pinref part="J1X" gate="A4983$2" pin="GND$2"/>
-<wire x1="-119.38" y1="48.26" x2="-119.38" y2="55.88" width="0.2032" layer="91"/>
+<wire x1="-73.66" y1="33.02" x2="-81.28" y2="33.02" width="0.2032" layer="91"/>
+<wire x1="-81.28" y1="33.02" x2="-81.28" y2="27.94" width="0.2032" layer="91"/>
+<pinref part="J1X" gate="A4983$2" pin="GND$1"/>
+<wire x1="-73.66" y1="63.5" x2="-81.28" y2="63.5" width="0.2032" layer="91"/>
+<wire x1="-81.28" y1="63.5" x2="-81.28" y2="33.02" width="0.2032" layer="91"/>
+<junction x="-81.28" y="33.02"/>
+<wire x1="-81.28" y1="33.02" x2="-106.68" y2="33.02" width="0.2032" layer="91"/>
+<wire x1="-106.68" y1="33.02" x2="-106.68" y2="35.56" width="0.2032" layer="91"/>
+<pinref part="Q2" gate="G$1" pin="S"/>
 </segment>
+</net>
+<net name="N$1" class="0">
 <segment>
-<pinref part="J1X" gate="A4983$2" pin="GND$1"/>
-<pinref part="GND37" gate="1" pin="GND"/>
-<wire x1="-149.86" y1="55.88" x2="-149.86" y2="48.26" width="0.2032" layer="91"/>
+<pinref part="JP1" gate="A" pin="1"/>
+<pinref part="J1X" gate="A4983$1" pin="STEP"/>
+<wire x1="-132.08" y1="38.1" x2="-139.7" y2="38.1" width="0.2032" layer="91"/>
+</segment>
+</net>
+<net name="N$3" class="0">
+<segment>
+<wire x1="-116.84" y1="38.1" x2="-111.76" y2="38.1" width="0.2032" layer="91"/>
+<pinref part="Q2" gate="G$1" pin="G"/>
+<pinref part="R1" gate="G$1" pin="2"/>
+</segment>
+</net>
+<net name="N$2" class="0">
+<segment>
+<pinref part="JP1" gate="A" pin="2"/>
+<wire x1="-129.54" y1="38.1" x2="-127" y2="38.1" width="0.2032" layer="91"/>
+<pinref part="R1" gate="G$1" pin="1"/>
+</segment>
+</net>
+<net name="N$4" class="0">
+<segment>
+<pinref part="J1X" gate="A4983$2" pin="VMOT"/>
+<wire x1="-73.66" y1="68.58" x2="-88.9" y2="68.58" width="0.2032" layer="91"/>
+<wire x1="-88.9" y1="68.58" x2="-88.9" y2="58.42" width="0.2032" layer="91"/>
+<wire x1="-88.9" y1="58.42" x2="-96.52" y2="58.42" width="0.2032" layer="91"/>
+<pinref part="J1X" gate="A4983$2" pin="2B"/>
+<wire x1="-73.66" y1="58.42" x2="-88.9" y2="58.42" width="0.2032" layer="91"/>
+<junction x="-88.9" y="58.42"/>
+<pinref part="D1" gate="G$1" pin="C"/>
+</segment>
+</net>
+<net name="N$5" class="0">
+<segment>
+<pinref part="J1X" gate="A4983$2" pin="2A"/>
+<wire x1="-73.66" y1="53.34" x2="-88.9" y2="53.34" width="0.2032" layer="91"/>
+<pinref part="D1" gate="G$1" pin="A"/>
+<pinref part="Q2" gate="G$1" pin="D"/>
+<wire x1="-88.9" y1="53.34" x2="-96.52" y2="53.34" width="0.2032" layer="91"/>
+<wire x1="-106.68" y1="45.72" x2="-88.9" y2="45.72" width="0.2032" layer="91"/>
+<wire x1="-88.9" y1="53.34" x2="-88.9" y2="45.72" width="0.2032" layer="91"/>
+<junction x="-88.9" y="53.34"/>
 </segment>
 </net>
@@
 </sheet>
 </sheets>
+<errors>
+</errors>
 </schematic>
 </drawing>
